File: 6301-temp-sensor.kicad_pcb (KiCad board)
At the start: 2 copper layers, 18 parts, among them P101 CONN_01X15, P102 CONN_01X15, U101 MPQ3906, U102 MPQ3904, U103 4066, U104 TL074, U105 LM311N

Commit message: fixed schematic and layout
Parts:
- added R107: 10k, Resistors_ThroughHole:Resistor_Horizontal_RM10mm, F.Cu at (121.8, 102.8)
Connections:
- R103 pad 1: +3V3 -> /3.3V
Routing:
- net /3.3V: track 62.0 -> 87.1 mm
- net /5V: track 113.2 -> 117.9 mm
Other:
- board outline added: 92.8 x 51.4 mm

Commit message: More fixes
Connections:
- U101 pad 10: /3.3V -> /3.0V
- U101 pad 3: /3.3V -> /3.0V
Routing:
- net /3.0V: track 36.0 -> 111.2 mm, vias 0 -> 1
- net /3.3V: track 87.1 -> 49.8 mm
Changed lines of the file:
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@@
   (general
     (links 50)
-    (no_connects 3)
+    (no_connects 1)
     (area 40.424999 72.824999 133.375001 124.375001)
     (thickness 1.6)
     (drawings 6)
-    (tracks 148)
+    (tracks 149)
     (zones 0)
     (modules 19)
@@
       (net 38 "Net-(U101-Pad2)"))
     (pad 3 thru_hole oval (at 0 5.08) (size 1.6 1.6) (drill 0.8) (layers *.Cu *.Mask F.SilkS)
-      (net 3 /3.3V))
+      (net 5 /3.0V))
     (pad 4 thru_hole oval (at 0 7.62) (size 1.6 1.6) (drill 0.8) (layers *.Cu *.Mask F.SilkS)
       (net 39 "Net-(U101-Pad4)"))
@@
       (net 38 "Net-(U101-Pad2)"))
     (pad 10 thru_hole oval (at 7.62 10.16) (size 1.6 1.6) (drill 0.8) (layers *.Cu *.Mask F.SilkS)
-      (net 3 /3.3V))
+      (net 5 /3.0V))
     (pad 11 thru_hole oval (at 7.62 7.62) (size 1.6 1.6) (drill 0.8) (layers *.Cu *.Mask F.SilkS)
       (net 41 "Net-(U101-Pad11)"))
@@
   (segment (start 74 99.08) (end 74 104.3) (width 0.25) (layer F.Cu) (net 3))
   (segment (start 88.9 107.0864) (end 88.9 106.934) (width 0.25) (layer F.Cu) (net 3))
-  (segment (start 65.7 112.1) (end 61.956 115.844) (width 0.25) (layer F.Cu) (net 3))
-  (segment (start 61.956 115.844) (end 59.12 115.844) (width 0.25) (layer F.Cu) (net 3))
-  (segment (start 65.7 104.3) (end 65.7 112.1) (width 0.25) (layer F.Cu) (net 3))
-  (segment (start 70.92 99.08) (end 65.7 104.3) (width 0.25) (layer F.Cu) (net 3))
-  (segment (start 74 99.08) (end 70.92 99.08) (width 0.25) (layer F.Cu) (net 3))
-  (segment (start 59.919999 115.044001) (end 59.12 115.844) (width 0.25) (layer F.Cu) (net 3))
   (segment (start 88.9 106.7816) (end 88.9 106.934) (width 0.25) (layer F.Cu) (net 3))
-  (segment (start 59.12 115.844) (end 56.58 115.844) (width 0.25) (layer F.Cu) (net 3))
-  (segment (start 56.58 115.844) (end 51.5 110.764) (width 0.25) (layer F.Cu) (net 3))
   (segment (start 59.1 87.38) (end 51.48 87.38) (width 0.25) (layer F.Cu) (net 4))
   (segment (start 53.676 123.1) (end 64.9 123.1) (width 0.25) (layer B.Cu) (net 4))
@@
   (segment (start 123.094 82.46) (end 123.094 81.32863) (width 0.25) (layer F.Cu) (net 4))
   (segment (start 111.08 90.08) (end 111 90) (width 0.25) (layer F.Cu) (net 4))
+  (segment (start 66.3 83.7) (end 83.94 83.7) (width 0.25) (layer B.Cu) (net 5))
+  (segment (start 83.94 83.7) (end 90.932 76.708) (width 0.25) (layer B.Cu) (net 5))
+  (segment (start 61.956 115.844) (end 66.3 111.5) (width 0.25) (layer F.Cu) (net 5))
+  (segment (start 66.3 111.5) (end 66.3 83.7) (width 0.25) (layer F.Cu) (net 5))
+  (via (at 66.3 83.7) (size 0.6) (drill 0.4) (layers F.Cu B.Cu) (net 5))
+  (segment (start 61.956 115.844) (end 59.12 115.844) (width 0.25) (layer F.Cu) (net 5))
+  (segment (start 59.919999 115.044001) (end 59.12 115.844) (width 0.25) (layer F.Cu) (net 5))
+  (segment (start 59.12 115.844) (end 56.58 115.844) (width 0.25) (layer F.Cu) (net 5))
+  (segment (start 56.58 115.844) (end 51.5 110.764) (width 0.25) (layer F.Cu) (net 5))
   (segment (start 105.7 92.76) (end 105.7 89.78) (width 0.25) (layer F.Cu) (net 5))
   (segment (start 105.7 89.78) (end 103.38 87.46) (width 0.25) (layer F.Cu) (net 5))
