File: 6301-temp-sensor.sch (KiCad schematic (older format))
At the start: 16 parts, among them P101 CONN_01X15, P102 CONN_01X15, U101 MPQ3906, U102 MPQ3904, U103 4066, U104 TL074, U105 LM311N

Commit message: fixed schematic and layout
Parts:
- added R107: 10k, Resistors_ThroughHole:Resistor_Horizontal_RM10mm, symbol R
Connections:
- net +3V3 is gone; now on net 3.3V: R103.1
- net +5V is gone; now on net 5V: U104.4 (V+)
- net 5V: now also R107.1
- net at P101.5 (P5), R106.1, U105.7: now also R107.2
Changed lines of the file:
@@
-	1    0    0    -1
-$EndComp
-$Comp
-L +3.3V #PWR02
-U 1 1 584458B6
-P 6000 5400
-F 0 "#PWR02" H 6000 5250 50  0001 C CNN
-F 1 "+3.3V" H 6000 5540 50  0000 C CNN
-F 2 "" H 6000 5400 50  0000 C CNN
-F 3 "" H 6000 5400 50  0000 C CNN
-	1    6000 5400
 	1    0    0    -1
 $EndComp
@@
 5V
 $Comp
-L GND #PWR03
+L GND #PWR02
 U 1 1 58445C39
 P 6400 2850
-F 0 "#PWR03" H 6400 2600 50  0001 C CNN
+F 0 "#PWR02" H 6400 2600 50  0001 C CNN
 F 1 "GND" H 6400 2700 50  0000 C CNN
 F 2 "" H 6400 2850 50  0000 C CNN
@@
 $EndComp
 $Comp
-L GND #PWR04
+L GND #PWR03
 U 1 1 58445C62
 P 4600 3500
-F 0 "#PWR04" H 4600 3250 50  0001 C CNN
+F 0 "#PWR03" H 4600 3250 50  0001 C CNN
 F 1 "GND" H 4600 3350 50  0000 C CNN
 F 2 "" H 4600 3500 50  0000 C CNN
@@
 $EndComp
 $Comp
-L GND #PWR05
+L GND #PWR04
 U 1 1 58449E51
 P 6850 6200
-F 0 "#PWR05" H 6850 5950 50  0001 C CNN
+F 0 "#PWR04" H 6850 5950 50  0001 C CNN
 F 1 "GND" H 6850 6050 50  0000 C CNN
 F 2 "" H 6850 6200 50  0000 C CNN
 F 3 "" H 6850 6200 50  0000 C CNN
 	1    6850 6200
-	1    0    0    -1
-$EndComp
-$Comp
-L +5V #PWR06
-U 1 1 58449E7D
-P 6850 5350
-F 0 "#PWR06" H 6850 5200 50  0001 C CNN
-F 1 "+5V" H 6850 5490 50  0000 C CNN
-F 2 "" H 6850 5350 50  0000 C CNN
-F 3 "" H 6850 5350 50  0000 C CNN
-	1    6850 5350
 	1    0    0    -1
 $EndComp
@@
 $EndComp
 $Comp
-L GND #PWR07
+L GND #PWR05
 U 1 1 5844A4F0
 P 8900 6300
-F 0 "#PWR07" H 8900 6050 50  0001 C CNN
+F 0 "#PWR05" H 8900 6050 50  0001 C CNN
 F 1 "GND" H 8900 6150 50  0000 C CNN
 F 2 "" H 8900 6300 50  0000 C CNN
@@
 $EndComp
 $Comp
-L GND #PWR08
+L GND #PWR06
 U 1 1 5844A5D3
 P 9550 6300
-F 0 "#PWR08" H 9550 6050 50  0001 C CNN
+F 0 "#PWR06" H 9550 6050 50  0001 C CNN
 F 1 "GND" H 9550 6150 50  0000 C CNN
 F 2 "" H 9550 6300 50  0000 C CNN
@@
 5V
 $Comp
-L GND #PWR010
+L GND #PWR07
 U 1 1 5844AFDF
 P 10800 2850
-F 0 "#PWR010" H 10800 2600 50  0001 C CNN
+F 0 "#PWR07" H 10800 2600 50  0001 C CNN
 F 1 "GND" H 10800 2700 50  0000 C CNN
 F 2 "" H 10800 2850 50  0000 C CNN
@@
 NoConn ~ 8600 3300
 $Comp
-L GND #PWR011
+L GND #PWR08
 U 1 1 5844B1E0
 P 8300 3700
-F 0 "#PWR011" H 8300 3450 50  0001 C CNN
+F 0 "#PWR08" H 8300 3450 50  0001 C CNN
 F 1 "GND" H 8300 3550 50  0000 C CNN
 F 2 "" H 8300 3700 50  0000 C CNN
@@
 $EndComp
 $Comp
-L GND #PWR012
+L GND #PWR09
 U 1 1 5844EE1F
 P 1200 4000
-F 0 "#PWR012" H 1200 3750 50  0001 C CNN
+F 0 "#PWR09" H 1200 3750 50  0001 C CNN
 F 1 "GND" H 1200 3850 50  0000 C CNN
 F 2 "" H 1200 4000 50  0000 C CNN
@@
 	8200 2600 8200 2900
 Wire Wire Line
-	8300 3700 8300 3500
+	8300 3500 8300 3700
 Wire Wire Line
 	8600 3200 9450 3200
@@
 	3100 4950 3100 5000
 $Comp
-L GND #PWR013
+L GND #PWR010
 U 1 1 5844F02B
 P 3100 5000
-F 0 "#PWR013" H 3100 4750 50  0001 C CNN
+F 0 "#PWR010" H 3100 4750 50  0001 C CNN
 F 1 "GND" H 3100 4850 50  0000 C CNN
 F 2 "" H 3100 5000 50  0000 C CNN
@@
 $EndComp
 $Comp
-L GND #PWR014
+L GND #PWR011
 U 1 1 5844F078
 P 1200 5000
-F 0 "#PWR014" H 1200 4750 50  0001 C CNN
+F 0 "#PWR011" H 1200 4750 50  0001 C CNN
 F 1 "GND" H 1200 4850 50  0000 C CNN
 F 2 "" H 1200 5000 50  0000 C CNN
@@
 	1400 6600 1400 6700
 $Comp
-L GND #PWR015
+L GND #PWR012
 U 1 1 5844F562
 P 1400 6700
-F 0 "#PWR015" H 1400 6450 50  0001 C CNN
+F 0 "#PWR012" H 1400 6450 50  0001 C CNN
 F 1 "GND" H 1400 6550 50  0000 C CNN
 F 2 "" H 1400 6700 50  0000 C CNN
@@
 NoConn ~ 9700 2750
 NoConn ~ 9700 2850
+Text Label 6850 5350 0    60   ~ 0
+5V
+Text Label 6000 5400 0    60   ~ 0
+3.3V
+$Comp
+L R R107
+U 1 1 584CD30D
+P 9100 2800
+F 0 "R107" V 9180 2800 50  0000 C CNN
+F 1 "10k" V 9100 2800 50  0000 C CNN
+F 2 "Resistors_ThroughHole:Resistor_Horizontal_RM10mm" V 9030 2800 50  0001 C CNN
+F 3 "" H 9100 2800 50  0000 C CNN
+	1    9100 2800
+	1    0    0    -1
+$EndComp
+Wire Wire Line
+	9100 2950 9100 3200
+Connection ~ 9100 3200
+Wire Wire Line
+	9100 2650 9100 2500
+Text Label 9100 2500 0    60   ~ 0
+5V
 $EndSCHEMATC

Commit message: More fixes
Connections:
- net 3.0V: now also U101.10 (E3), U101.3 (E1)
- net 3.3V: no longer U101.10 (E3), U101.3 (E1)
Changed lines of the file:
@@
 encoding utf-8
 Sheet 1 1
-Title ""
+Title "Temperature Sensor"
 Date ""
 Rev ""
-Comp ""
+Comp "Jimmy Mawdsley, MIT"
 Comment1 ""
 Comment2 ""
@@
 Connection ~ 2200 2300
 Text Label 2200 2050 0    60   ~ 0
-3.3V
+3.0V
 Connection ~ 1400 3550
 NoConn ~ 10550 2750
